File: hardware/dac_ino_lite/dac_ino.kicad_pcb (KiCad board)
At the start: 2 copper layers, 64 x 55.5 mm, 23 parts, among them J1 CV OUT A, J2 CV OUT B, J5 GATE OUT A, J6 Conn_01x04, J7 Conn_01x04, J8 VCC, J9 Vin, Q1 2N3904, U1 MCP4922

Commit message: Name change
Parts:
- added G***: LOGO, dac_ino:analogoutput2, F.Cu at (178.0, 104.7)
- added G***: LOGO, dac_ino:deco2, F.Cu at (143.4, 115.6)
Other:
- board text added: "DAC/INO"
- board text added: "dac/ino Vincenzo Pacella Rich Holmes 3/2020 cc-by-sa"
- board text removed: "dacarduino Vincenzo Pacella Rich Holmes 3/2020 cc-by-sa"
